File: PDM 2021.sch (EAGLE design)
At the start: 28 parts

Commit message: Add files via upload
Parts:
- added K1: SR4M4012, SR4M4012:SR4M4012
- added Q1: SI7336ADP-T1-GE3, SI7336ADP-T1-GE3:SI7336ADP-T1-GE3
- added R10, R11: (no value), rcl:R-US_R0805
Connections:
- new net GND: Q1.S_1, Q1.S_2, Q1.S_3, R11.1
- new net N$11: Q1.G, R10.1, R11.2
- new net N$12: K1.A1, Q1.D_1, Q1.D_2, Q1.D_3, Q1.D_4
- new net N$14: CH11.1A, CH11.1B, K1.24, K1.34, K1.44, R9.1
- net CH11: now also K1.23, K1.33, K1.43, K1.A2, R10.2; no longer CH11.1A, CH11.1B, R9.1

Commit message: Add files via upload
Parts:
- removed CH11, CH3: 3568FUSEHOLDER, ACC-MB-R0:3568FUSEHOLDER
- removed K1: SR4M4012, SR4M4012:SR4M4012
- removed LED3, LED9: (no value), led:LEDCHIP-LED0805
- removed Q1: SI7336ADP-T1-GE3, SI7336ADP-T1-GE3:SI7336ADP-T1-GE3
- removed R3, R9: (no value), rcl:R-US_R0805
- added R12, R13, R14, R15, R16: (no value), rcl:R-US_R0805
- added U$1, U$10, U$2, U$3, U$5, U$7, U$8, U$9: _CUSTOM_111_CUSTOM_SQJ407EP-T1_GE3, ACC-MB-R0:_CUSTOM_111_CUSTOM_SQJ407EP-T1_GE3
- added U$11, U$12, U$6: RK7002BMT116, ACC-MB-R0:RK7002BMT116
Connections:
- removed net CH1: CH1.1A, CH1.1B, R1.1, U$4.P$18, U$4.P$19
- removed net CH3: CH3.1A, CH3.1B, R3.1, U$4.P$16, U$4.P$21
- removed net COMMON: CH1.2A, CH1.2B, CH11.2A, CH11.2B, CH2.2A, CH2.2B, CH3.2A, CH3.2B, CH4.2A, CH4.2B, CH5.2A, CH5.2B, CH6.2A, CH6.2B, CH7.2A, CH7.2B, CH9.2A, CH9.2B, LED1.C, LED2.C, LED3.C, LED4.C, LED5.C, LED6.C, LED7.C, LED8.C, LED9.C
- removed net N$12: K1.A1, Q1.D_1, Q1.D_2, Q1.D_3, Q1.D_4
- new net N$10: R10.1, R11.2, U$6.G
- new net N$13: R16.2, U$11.D, U$7.G, U$8.G
- new net N$16: R10.2, R12.2, U$1.S, U$2.S, U$3.S, U$4.P$1, U$4.P$11, U$4.P$12, U$4.P$2, U$5.S
- new net N$17: R15.2, U$10.G, U$12.D, U$9.G
- new net N$19: R14.2, U$12.G, U$4.P$16
- new net N$9: CH1.2A, LED1.C, U$7.D, U$8.D
- net CH11: now also CH2.2A, CH2.2B, LED2.C, U$10.D, U$9.D; no longer K1.23, K1.33, K1.43, K1.A2, R10.2, U$4.P$1, U$4.P$11, U$4.P$12, U$4.P$2
- net CH8: no longer U$4.P$6, U$4.P$7
- net GND: now also R13.1, R14.1, U$11.S, U$12.S, U$4.P$6, U$4.P$7, U$6.S; no longer Q1.S_1, Q1.S_2, Q1.S_3
- net N$1: now also CH4.2A, CH4.2B, CH5.2A, CH5.2B, CH6.2A, CH6.2B, CH7.2A, CH7.2B, CH9.2A, CH9.2B, LED4.C, LED5.C, LED6.C, LED7.C, LED8.C, R15.1, R16.1, U$1.D, U$10.S, U$2.D, U$3.D, U$5.D, U$7.S, U$8.S, U$9.S; no longer LED9.A, R9.2
- net N$11: now also R12.1, U$1.G, U$2.G, U$3.G, U$5.G, U$6.D; no longer Q1.G, R10.1, R11.2
- net N$14: now also R13.2, U$11.G, U$4.P$21; no longer CH11.1A, CH11.1B, K1.24, K1.34, K1.44, R9.1
- net N$7: now also CH1.1A, R1.1, U$4.P$18, U$4.P$19; no longer LED3.A, R3.2
Other:
- moved on the sheet: CH1, CH2, LED1, LED2, R1, R10, R11, R2
